File: hardware/kicad/redundant12v/redundant12v.kicad_pcb (KiCad board)
At the start: 2 copper layers, 67.1 x 26.4 mm, 28 parts, among them J1 Conn_01x07, J2 IDC 2x5 Male, U1 ATTINY212-SSF, U2 TI MAX232EID, U3 LD1117S50CTR, X1 ECS-3951M-018-AU-TR

Commit message: Resistors R1, R2 are now 47K
Parts:
- R1, R2: value 10K -> 47K
Changed lines of the file:
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@@
       (effects (font (size 1 1) (thickness 0.15)))
     )
-    (fp_text value "10K" (at 0 1.65 90) (layer "F.Fab")
+    (fp_text value "47K" (at 0 1.65 90) (layer "F.Fab")
       (effects (font (size 1 1) (thickness 0.15)))
     )
@@
       (effects (font (size 1 1) (thickness 0.15)))
     )
-    (fp_text value "10K" (at 0.127 3.936 90) (layer "F.Fab")
+    (fp_text value "47K" (at 0.127 3.936 90) (layer "F.Fab")
       (effects (font (size 1 1) (thickness 0.15)))
     )
